File: electronics/mainboard.brd (EAGLE design)
At the start: 160 x 160 mm, 18 parts, among them T1 NPN_BC817,215

Commit message: Board wip
Parts:
- added U$5: BOOSTER, rhoban:BOOSTER_390V
- added U$6, U$7, U$8, U$9: (no value), SparkFun-Hardware:STAND-OFF
- added XT60: CONNEC_ALIM, rhoban:XT60
- moved REG5V 121.1 mm to (47.8, -39.1), turned to 270 degrees
- moved REG3.3V 117.2 mm to (47.8, -26.4), turned to 270 degrees
- moved BOOSTER 105.8 mm to (70.6, -21.6), turned to 90 degrees
- moved SOLENOID 105.0 mm to (70.6, 20.3), turned to 90 degrees
- moved POWERCAP2 101.6 mm to (70.6, -6.35), turned to 90 degrees
- moved POWERCAP1 101.3 mm to (70.6, 5.08), turned to 90 degrees
- moved U$4 101.3 mm to (42.9, -45.5), turned to 270 degrees
- moved U$3 94.8 mm to (42.9, -32.8), turned to 270 degrees
- moved U$1 89.3 mm to (60.5, 15.2), turned to 0 degrees
- moved R3 78.3 mm to (52.6, 16.0), turned to 90 degrees
- moved T1 76.7 mm to (52.6, 10.9), turned to 0 degrees
- moved R1 73.9 mm to (51.3, 5.84), turned to 90 degrees
- moved R2 71.9 mm to (50.0, 2.03), turned to 180 degrees
- moved U$2 57.0 mm to (-25.9, 55.6)
- moved U$12 55.2 mm to (-39.9, 45.7)
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Connections:
- net GND: now also U$5.IN-, U$5.OUT-, XT60.GND
- net VBOOST: now also U$5.OUT+
- net VIN: now also U$5.VIN, XT60.V+
Other:
- board size 160 x 160 mm -> 170 x 170 mm

Commit message: wip
Parts:
- added C1: (no value), rcl:EB30D
Changed lines of the file:
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@@
 <element name="U$8" library="SparkFun-Hardware" package="STAND-OFF" value="" x="-57.904" y="-57.842"/>
 <element name="U$9" library="SparkFun-Hardware" package="STAND-OFF" value="" x="57.846" y="-58.092"/>
+<element name="C1" library="rcl" package="EB30D" value="" x="-68" y="-102"/>
 </elements>
 <signals>

Commit message: Infrared barrier
Parts:
- removed C1: (no value), rcl:EB30D
- added EMIT, RECEIVE: CONNEC_1X02JST-ZH, rhoban:JST_ZH_2P
- added R4: 1K, rhoban:R0805
- added R5: 36, rhoban:R0805
- added R6: 10K, rhoban:R0805
- added T2: NPN_BC817,215, rhoban:SOT-23
- moved U$13 23.5 mm to (-54.0, 46.0)
- moved R8 23.5 mm to (-67.4, 45.7)
- moved U$12 23.5 mm to (-63.4, 45.7)
- moved U$2 13.0 mm to (-27.0, 42.6)
Connections:
- new net IR_EMIT: MAPLE.X12, R4.1
- new net IR_RECEIVE: MAPLE.X10, R6.2, RECEIVE.P$1
- new net N$11: R4.2, T2.1
- new net N$6: EMIT.P$1, R5.2
- new net N$7: EMIT.P$2, T2.3
- net 3.3: now also R6.1
- net GND: now also RECEIVE.P$2, T2.2
- net VCC: now also R5.1
Other:
- board text added: "LONG"
- board text added: "SHORT"

Commit message: Electronics wip
Parts:
- removed BOOSTER: CONNEC_1X03BIG, rhoban:CONNEC_1X03_BIG
- added COM1, COM2, COM3: NRF24L01, rhoban:NRF24L01
- added U$10: LS7366RSO14, rhoban:SO14
- moved POWERCAP2 146.2 mm to (-72.6, -35.3), turned to 0 degrees
- moved POWERCAP1 137.4 mm to (-60.7, -35.3), turned to 0 degrees
- moved U$1 133.2 mm to (-58.4, -45.0), turned to 270 degrees
- moved SOLENOID 131.2 mm to (-48.3, -35.3), turned to 0 degrees
- moved T1 112.9 mm to (-45.0, -46.0), turned to 90 degrees
- moved R1 110.3 mm to (-43.2, -51.1)
- moved R2 109.5 mm to (-45.7, -51.1), turned to 270 degrees
- moved R3 109.3 mm to (-41.1, -40.1), turned to 0 degrees
- moved U$2 82.5 mm to (53.1, 22.9), turned to 0 degrees
- moved R8 42.7 mm to (-26.9, 59.1), turned to 0 degrees
- moved U$12 40.4 mm to (-26.9, 63.1), turned to 0 degrees
- moved U$13 37.7 mm to (-27.2, 72.5), turned to 90 degrees
- moved REG3.3V 25.7 mm to (61.7, -4.83)
- moved U$3 25.4 mm to (55.9, -10.9)
- moved REG5V 25.3 mm to (61.7, -18.0)
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Connections:
- removed net N$10: U$3.-
- net GND: now also U$3.-; no longer BOOSTER.P$1
- net VBOOST: no longer BOOSTER.P$3
- net VIN: no longer BOOSTER.P$2

Commit message: Electronics wip
Parts:
- removed U$6, U$7, U$8, U$9: (no value), SparkFun-Hardware:STAND-OFF
- added R10, R11, R12, R13, R14, R15, R7, R9: 3K, rhoban:R0805
- added U1: CD4051BM, rhoban:SOIC127P600X175-16N
- added X1, X2, X3, X4, X5: JST-XH-10-PIN-LONG-PAD, Rembrandt Electronics - JST XH Connectors v1-0:JST-XH-10-PACKAGE-LONG-PAD
- moved XT60 121.7 mm to (-49.8, -66.3), turned to 0 degrees
- moved RECEIVE 118.2 mm to (67.8, 42.2), turned to 270 degrees
- moved EMIT 117.4 mm to (71.8, 34.2), turned to 270 degrees
- moved R6 112.9 mm to (63.9, 41.3), turned to 270 degrees
- moved U$13 112.5 mm to (73.8, 22.9), turned to 0 degrees
- moved T2 111.1 mm to (66.3, 34.9), turned to 270 degrees
- moved R5 109.0 mm to (66.4, 31.7), turned to 0 degrees
- moved R4 107.5 mm to (63.1, 35.3), turned to 90 degrees
- moved COM1 105.5 mm to (-19.1, 54.1), turned to 90 degrees
- moved U$12 100.5 mm to (65.2, 22.9), turned to 270 degrees
- moved R8 95.9 mm to (61.8, 22.9), turned to 270 degrees
- moved REG3.3V 94.6 mm to (-28.4, -33.3)
- moved REG5V 94.6 mm to (-28.4, -46.5)
- moved U$3 94.6 mm to (-34.3, -39.4)
- moved U$4 94.6 mm to (-34.0, -52.6)
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Connections:
- new net CS1: R7.2, U1.13
- new net CS2: R9.2, U1.14
- new net CS3: R10.2, U1.15
- new net CS4: R11.2, U1.12
- new net CS5: R12.2, U1.1
- new net CS6: R13.2, U1.5
- new net CS7: R14.2, U1.2
- new net CS8: R15.2, U1.4
- new net CSA1: U1.11
- new net CSA2: U1.10
- new net CSA3: U1.9
- net 3.3: now also R10.1, R11.1, R12.1, R13.1, R14.1, R15.1, R7.1, R9.1, U1.16
- net GND: now also U1.3, U1.6, U1.7, U1.8

Commit message: Maxon controllers (wip)
Parts:
- added C1, C17, C18, C2, C3, C4, C5, C6: 15pF, rhoban:C0603
- added ENC1, ENC2, ENC3, ENC4: LS7366RSO14, rhoban:SO14
- added R16, R17, R19, R20, R22, R23, R25, R26, R28, R29: 1K, rhoban:R0805
- added R18, R21, R24, R27, R30: 24k, rhoban:R0805
- added U$6, U$7, U$8, U$9: MAXON380200, rhoban:MAXON380200
- added XTAL1, XTAL2, XTAL3, XTAL4: 40Mhz, rhoban:HC49US
- R5: value 36 -> 60
- U$10: value LS7366RSO14 -> MAXON380200; device rhoban:SO14 -> rhoban:MAXON380200
- moved U$10 40.3 mm to (70.4, 10.4), turned to 180 degrees
- moved X1 14.2 mm to (-5.33, 74.2)
- moved X3 8.62 mm to (-11.7, -76.7), turned to 0 degrees
- moved X2 3.70 mm to (24.4, 73.7)
- moved X4 1.48 mm to (17.5, -76.5), turned to 0 degrees
- moved X5 0.57 mm to (78.5, 0.51), turned to 90 degrees
Connections:
- new net INDEX: ENC1.10, ENC2.10, ENC3.10, ENC4.10
- new net M1_A: ENC1.12, X1.9
- new net M1_B: ENC1.11, X1.10
- new net M1_DIR: U$6.23
- new net M1_HALL1: U$6.13, X1.6
- new net M1_HALL2: U$6.15, X1.7
- new net M1_HALL3: U$6.17, X1.8
- new net M1_SPEED: U$6.26
- new net M1_W1: U$6.1, U$6.2, X1.1
- new net M1_W2: U$6.3, U$6.4, X1.2
- new net M1_W3: U$6.5, U$6.6, X1.3
- new net M2_A: ENC2.12, X2.9
- new net M2_B: ENC2.11, X2.10
- new net M2_DIR: U$7.23
- new net M2_HALL1: U$7.13, X2.6
- new net M2_HALL2: U$7.15, X2.7
- new net M2_HALL3: U$7.17, X2.8
- new net M2_SPEED: U$7.26
- new net M2_W1: U$7.1, U$7.2, X2.1
- new net M2_W2: U$7.3, U$7.4, X2.2
- new net M2_W3: U$7.5, U$7.6, X2.3
- new net M3_A: ENC3.12, X3.9
- new net M3_B: ENC3.11, X3.10
- new net M3_DIR: U$8.23
- new net M3_HALL1: U$8.13, X3.6
- new net M3_HALL2: U$8.15, X3.7
- new net M3_HALL3: U$8.17, X3.8
- new net M3_SPEED: U$8.26
- new net M3_W1: U$8.1, U$8.2, X3.1
- new net M3_W2: U$8.3, U$8.4, X3.2
- new net M3_W3: U$8.5, U$8.6, X3.3
- new net M4_A: ENC4.12, X4.9
- new net M4_B: ENC4.11, X4.10
- new net M4_DIR: U$9.23
- new net M4_HALL1: U$9.13, X4.6
- new net M4_HALL2: U$9.15, X4.7
- new net M4_HALL3: U$9.17, X4.8
- new net M4_SPEED: U$9.26
- new net M4_W1: U$9.1, U$9.2, X4.1
- new net M4_W2: U$9.3, U$9.4, X4.2
- new net M4_W3: U$9.5, U$9.6, X4.3
- new net M5_DIR: U$10.23
- new net M5_HALL1: U$10.13, X5.6
- new net M5_HALL2: U$10.15, X5.7
- new net M5_HALL3: U$10.17
- new net M5_SPEED: U$10.26
- new net M5_W1: U$10.1, U$10.2, X5.1
- new net M5_W2: U$10.3, U$10.4, X5.2
- new net M5_W3: U$10.5, U$10.6, X5.3
- new net MISO: ENC1.6, ENC2.6, ENC3.6, ENC4.6
- new net MOSI: ENC1.7, ENC2.7, ENC3.7, ENC4.7
- new net MOTORS_EN: U$10.22, U$6.22, U$7.22, U$8.22, U$9.22
- new net MT_HALL3: X5.8
- new net N$10: R16.2, U$6.20
- new net N$12: R17.2, U$6.21
- new net N$13: C1.2, ENC2.1, XTAL2.2
- new net N$14: C2.2, ENC2.2, XTAL2.1
- new net N$15: R19.2, U$7.20
- new net N$16: R18.2, U$6.25
- new net N$18: R20.2, U$7.21
- new net N$19: C17.2, ENC1.1, XTAL1.2
- new net N$20: C18.2, ENC1.2, XTAL1.1
- new net N$21: R21.2, U$7.25
- new net N$22: C3.2, ENC3.1, XTAL3.2
- new net N$23: C4.2, ENC3.2, XTAL3.1
- new net N$24: R22.2, U$8.20
- new net N$25: R23.2, U$8.21
- new net N$26: R24.2, U$8.25
- new net N$27: C5.2, ENC4.1, XTAL4.2
- new net N$28: C6.2, ENC4.2, XTAL4.1
- new net N$29: R25.2, U$9.20
- new net N$30: R26.2, U$9.21
- new net N$31: R27.2, U$9.25
- new net N$32: R28.2, U$10.20
- new net N$33: R29.2, U$10.21
- new net N$34: R30.2, U$10.25
- new net SCK: ENC1.5, ENC2.5, ENC3.5, ENC4.5
- net CS1: now also ENC1.4
- net CS2: now also ENC2.4
- net CS3: now also ENC3.4
- net CS4: now also ENC4.4
- net GND: now also C1.1, C17.1, C18.1, C2.1, C3.1, C4.1, C5.1, C6.1, ENC1.3, ENC2.3, ENC3.3, ENC4.3, R16.1, R18.1, R19.1, R21.1, R22.1, R24.1, R25.1, R27.1, R28.1, R30.1, U$10.10, U$10.14, U$10.16, U$10.24, U$10.9, U$6.10, U$6.14, U$6.16, U$6.24, U$6.9, U$7.10, U$7.14, U$7.16, U$7.24, U$7.9, U$8.10, U$8.14, U$8.16, U$8.24, U$8.9, U$9.10, U$9.14, U$9.16, U$9.24, U$9.9, X1.4, X2.4, X3.4, X4.4, X5.4
- net VCC: now also ENC1.14, ENC2.14, ENC3.14, ENC4.14, R17.1, R20.1, R23.1, R26.1, R29.1, U$10.11, U$6.11, U$7.11, U$8.11, U$9.11, X1.5, X2.5, X3.5, X4.5, X5.5; no longer R5.1
- net VIN: now also R5.1, U$10.7, U$10.8, U$6.7, U$6.8, U$7.7, U$7.8, U$8.7, U$8.8, U$9.7, U$9.8

Commit message: Routing ready board
Parts:
- removed SOLENOID: CONNEC_1X02BIG, rhoban:CONNEC_1X02_BIG
- added R31: 1K, rhoban:R0805
- added R32, R33: 3K, rhoban:R0805
- added SOLENOID1, SOLENOID2: CONNEC_1X02BIG, rhoban:CONNEC_1X02_BIG
- added T3: NPN_BC817,215, rhoban:SOT-23
- added U$11: TO-247A, to-247_n-channel_igbt:TO-247
- moved U$4 58.9 mm to (12.1, -15.9)
- moved U$3 58.8 mm to (12.1, -3.17)
- moved REG3.3V 57.9 mm to (16.5, 3.17)
- moved REG5V 57.8 mm to (16.5, -10.2)
- moved COM3 44.7 mm to (54.0, -19.1), turned to 180 degrees
- moved COM2 40.4 mm to (47.0, 20.3), turned to 0 degrees
- moved XT60 23.8 mm to (-27.7, -75.2), turned to 90 degrees
- moved R1 14.8 mm to (-31.1, -42.5), turned to 270 degrees
- moved T1 14.7 mm to (-33.0, -37.5)
- moved R2 14.2 mm to (-34.3, -42.5)
- moved R3 10.4 mm to (-33.0, -33.7)
- moved U$1 10.3 mm to (-48.3, -43.2)
- moved R23 8.60 mm to (-3.81, -54.0)
- moved XTAL3 8.57 mm to (-14.0, -50.2)
- moved R11 8.36 mm to (5.08, -15.2)
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Connections:
- removed net KICK: MAPLE.X3, R1.1, R2.1
- new net IRQ1: COM1.IRQ, MAPLE.X23
- new net IRQ2: COM2.IRQ, MAPLE.X24
- new net IRQ3: COM3.IRQ, MAPLE.X25
- new net KICK1: MAPLE.X7, R1.1, R2.1
- new net KICK2: MAPLE.X6, R31.1, R32.1
- new net N$17: R31.2, T3.1
- new net N$35: R33.1, T3.3, U$11.P$1
- new net N$36: SOLENOID2.P$2, U$11.P$2
- net 3.3: now also COM1.CE, COM1.VCC, COM2.CE, COM2.VCC, COM3.CE, COM3.VCC, R32.2
- net CS5: now also COM1.CSN
- net CS6: now also COM2.CSN
- net CS7: now also COM3.CSN
- net CSA1: now also MAPLE.X20
- net CSA2: now also MAPLE.X21
- net CSA3: now also MAPLE.X22
- net GND: now also COM1.GND, COM2.GND, COM3.GND, T3.2, U$11.P$3
- net INDEX: now also MAPLE.X26
- net M1_DIR: now also MAPLE.X13
- net M1_SPEED: now also MAPLE.X3
- net M2_DIR: now also MAPLE.X14
- net M2_SPEED: now also MAPLE.X4
- net M3_DIR: now also MAPLE.X17
- net M3_SPEED: now also MAPLE.X5
- net M4_DIR: now also MAPLE.X18
- net M4_SPEED: now also MAPLE.X8
- net M5_DIR: now also MAPLE.X19
- net M5_SPEED: now also MAPLE.X9
- net MISO: now also COM1.MISO, COM2.MISO, COM3.MISO, MAPLE.X29
- net MOSI: now also COM1.MOSI, COM2.MOSI, COM3.MOSI, MAPLE.X28
- net N$2: now also SOLENOID1.P$2; no longer SOLENOID.P$2
- net SCK: now also COM1.SCK, COM2.SCK, COM3.SCK, MAPLE.X30
- net VBOOST: now also SOLENOID1.P$1, SOLENOID2.P$1; no longer SOLENOID.P$1
- net VIN: now also R33.2
Routing:
- net GND: track 0.00 -> 10.6 mm, vias 0 -> 4

Commit message: SSL mainboard wip
Parts:
- added U$14, U$16, U$17, U$18: (no value), SparkFun-Hardware:STAND-OFF
- moved X2 127.4 mm to (-11.4, -49.5), turned to 0 degrees
- moved X1 127.1 mm to (-40.6, -49.5), turned to 0 degrees
- moved MAPLE 126.9 mm to (58.7, 55.3), turned to 270 degrees
- moved X5 118.2 mm to (-40.0, 5.08), turned to 0 degrees
- moved POWERCAP2 112.8 mm to (11.4, 42.5), turned to 180 degrees
- moved C1 112.6 mm to (-21.6, -36.2), turned to 180 degrees
- moved XT60 110.5 mm to (72.6, -28.8)
- moved U$6 110.2 mm to (-30.5, -42.5), turned to 90 degrees
- moved U$7 110.1 mm to (-1.27, -42.5), turned to 90 degrees
- moved RECEIVE 108.4 mm to (-37.5, 67.9), turned to 0 degrees
- moved C2 108.2 mm to (-17.1, -36.2), turned to 0 degrees
- moved R29 106.0 mm to (-40.6, 19.7), turned to 90 degrees
- moved C17 104.8 mm to (-50.2, -31.8), turned to 180 degrees
- moved U$10 103.5 mm to (-33.0, 13.3), turned to 90 degrees
- moved R6 103.4 mm to (-36.8, 64.1), turned to 0 degrees
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Routing:
- net GND: track 10.6 -> 18.7 mm, vias 4 -> 5
Other:
- board size 170 x 170 mm -> 158.8 x 159.4 mm
