File: electronics/mainboard.sch (EAGLE design)
At the start: 18 parts, among them T1 NPN_BC817,215

Commit message: Board wip
Parts:
- added U$5: BOOSTER, rhoban:BOOSTER
- added XT60: CONNEC_ALIM, rhoban:CONNEC_ALIM
Connections:
- net GND: now also U$5.IN-, U$5.OUT-, XT60.GND
- net VBOOST: now also U$5.OUT+
- net VIN: now also U$5.IN+, XT60.V+
Changed lines of the file:
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@@
 <part name="U$3" library="rhoban" deviceset="CPOL_EU" device="PANASONIC_D" value="47uF"/>
 <part name="U$4" library="rhoban" deviceset="CPOL_EU" device="PANASONIC_D" value="47uF"/>
+<part name="XT60" library="rhoban" deviceset="CONNEC_ALIM" device=""/>
+<part name="U$5" library="rhoban" deviceset="BOOSTER" device=""/>
 </parts>
 <sheets>
@@
 <instance part="U$3" gate="G$1" x="-190.5" y="73.66"/>
 <instance part="U$4" gate="G$1" x="-190.5" y="53.34"/>
+<instance part="XT60" gate="G$1" x="-165.1" y="99.06"/>
+<instance part="U$5" gate="G$1" x="-129.54" y="96.52"/>
 </instances>
 <busses>
@@
 <label x="-190.5" y="48.26" size="1.778" layer="95"/>
 </segment>
+<segment>
+<pinref part="XT60" gate="G$1" pin="GND"/>
+<wire x1="-170.18" y1="104.14" x2="-177.8" y2="104.14" width="0.1524" layer="91"/>
+<label x="-182.88" y="104.14" size="1.778" layer="95"/>
+</segment>
+<segment>
+<pinref part="U$5" gate="G$1" pin="OUT-"/>
+<wire x1="-104.14" y1="104.14" x2="-99.06" y2="104.14" width="0.1524" layer="91"/>
+<label x="-99.06" y="104.14" size="1.778" layer="95"/>
+</segment>
+<segment>
+<pinref part="U$5" gate="G$1" pin="IN-"/>
+<wire x1="-134.62" y1="104.14" x2="-139.7" y2="104.14" width="0.1524" layer="91"/>
+<label x="-147.32" y="104.14" size="1.778" layer="95"/>
+</segment>
 </net>
 <net name="N$4" class="0">
@@
 <wire x1="-160.02" y1="58.42" x2="-165.1" y2="58.42" width="0.1524" layer="91"/>
 <label x="-170.18" y="58.42" size="1.778" layer="95"/>
+</segment>
+<segment>
+<pinref part="XT60" gate="G$1" pin="V+"/>
+<wire x1="-170.18" y1="109.22" x2="-177.8" y2="109.22" width="0.1524" layer="91"/>
+<label x="-182.88" y="109.22" size="1.778" layer="95"/>
+</segment>
+<segment>
+<pinref part="U$5" gate="G$1" pin="IN+"/>
+<wire x1="-134.62" y1="111.76" x2="-139.7" y2="111.76" width="0.1524" layer="91"/>
+<label x="-147.32" y="111.76" size="1.778" layer="95"/>
 </segment>
 </net>
@@
 <junction x="38.1" y="78.74"/>
 </segment>
-</net>
+<segment>
+<pinref part="U$5" gate="G$1" pin="OUT+"/>
+<wire x1="-104.14" y1="111.76" x2="-99.06" y2="111.76" width="0.1524" layer="91"/>
+<label x="-99.06" y="111.76" size="1.778" layer="95"/>
+</segment>
+</net>

Commit message: wip
Parts:
- added C1: (no value), rcl:CPOL-USE10-30
Changed lines of the file:
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@@
 <part name="XT60" library="rhoban" deviceset="CONNEC_ALIM" device=""/>
 <part name="U$5" library="rhoban" deviceset="BOOSTER" device=""/>
+<part name="C1" library="rcl" deviceset="CPOL-US" device="E10-30"/>
 </parts>
 <sheets>
@@
 <instance part="XT60" gate="G$1" x="-165.1" y="99.06"/>
 <instance part="U$5" gate="G$1" x="-129.54" y="96.52"/>
+<instance part="C1" gate="G$1" x="-134.62" y="10.16"/>
 </instances>
 <busses>

Commit message: Infrared barrier
Parts:
- removed C1: (no value), rcl:CPOL-USE10-30
- added EMIT, RECEIVE: CONNEC_1X02JST-ZH, rhoban:CONNEC_1X02JST-ZH
- added R4: 1K, rhoban:RESISTANCE-R0805
- added R5: 36, rhoban:RESISTANCE-R0805
- added R6: 10K, rhoban:RESISTANCE-R0805
- added T2: NPN_BC817,215, rhoban:NPN_BC817,215
Connections:
- new net IR_EMIT: MAPLE.12, R4.1
- new net IR_RECEIVE: MAPLE.10, R6.2, RECEIVE.1
- new net N$11: R4.2, T2.B
- new net N$6: EMIT.1, R5.2
- new net N$7: EMIT.2, T2.C
- net 3.3: now also R6.1
- net GND: now also RECEIVE.2, T2.E
- net VCC: now also R5.1
Other:
- note added: "BUZZER"
- note added: "INFRARED"
- note added: "KICKER"
- note added: "MCU"
- note added: "POWER"
- moved on the sheet: BOOSTER, MAPLE, POWERCAP1, POWERCAP2, R1, R2, R3, R8, SOLENOID, T1, U$12

Commit message: Electronics wip
Parts:
- removed BOOSTER: CONNEC_1X03BIG, rhoban:CONNEC_1X03BIG
- added COM1, COM2, COM3: NRF24L01, rhoban:NRF24L01
- added U$10: LS7366RSO14, rhoban:LS7366RSO14
Connections:
- removed net N$10: U$3.-
- net GND: now also U$3.-; no longer BOOSTER.1
- net VBOOST: no longer BOOSTER.3
- net VIN: no longer BOOSTER.2
Other:
- note added: "COM"
- note added: "ENCODERS?"
Changed lines of the file:
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@@
 <part name="U$1" library="to-247_n-channel_igbt" deviceset="TO-247" device="A"/>
 <part name="SOLENOID" library="rhoban" deviceset="CONNEC_1X02" device="BIG"/>
-<part name="BOOSTER" library="rhoban" deviceset="CONNEC_1X03" device="BIG"/>
 <part name="POWERCAP2" library="rhoban" deviceset="CONNEC_1X02" device="BIG"/>
 <part name="POWERCAP1" library="rhoban" deviceset="CONNEC_1X02" device="BIG"/>
@@
 <part name="R5" library="rhoban" deviceset="RESISTANCE" device="-R0805" value="36"/>
 <part name="R6" library="rhoban" deviceset="RESISTANCE" device="-R0805" value="10K"/>
+<part name="U$10" library="rhoban" deviceset="LS7366R" device="SO14"/>
+<part name="COM1" library="rhoban" deviceset="NRF24L01" device=""/>
+<part name="COM2" library="rhoban" deviceset="NRF24L01" device=""/>
+<part name="COM3" library="rhoban" deviceset="NRF24L01" device=""/>
 </parts>
 <sheets>
@@
 <text x="30.48" y="106.68" size="6.4516" layer="95">KICKER</text>
 <text x="-182.88" y="-45.72" size="6.4516" layer="95">INFRARED</text>
+<text x="-48.26" y="-53.34" size="7.62" layer="104">ENCODERS?</text>
+<text x="55.88" y="-55.88" size="7.62" layer="104">COM</text>
 </plain>
 <instances>
@@
 <instance part="U$1" gate="G$1" x="60.96" y="38.1"/>
 <instance part="SOLENOID" gate="G$1" x="58.42" y="55.88"/>
-<instance part="BOOSTER" gate="G$1" x="58.42" y="88.9"/>
 <instance part="POWERCAP2" gate="G$1" x="58.42" y="66.04"/>
 <instance part="POWERCAP1" gate="G$1" x="58.42" y="76.2"/>
@@
 <instance part="R5" gate="G$1" x="-167.64" y="-55.88"/>
 <instance part="R6" gate="G$1" x="-167.64" y="-86.36"/>
+<instance part="U$10" gate="G$1" x="-20.32" y="-76.2"/>
+<instance part="COM1" gate="G$1" x="71.12" y="-78.74"/>
+<instance part="COM2" gate="G$1" x="71.12" y="-106.68"/>
+<instance part="COM3" gate="G$1" x="71.12" y="-137.16"/>
 </instances>
 <busses>
@@
 </segment>
 <segment>
-<pinref part="BOOSTER" gate="G$1" pin="1"/>
-<wire x1="60.96" y1="93.98" x2="53.34" y2="93.98" width="0.1524" layer="91"/>
-<label x="48.26" y="93.98" size="1.778" layer="95"/>
-</segment>
-<segment>
 <pinref part="POWERCAP2" gate="G$1" pin="1"/>
 <wire x1="60.96" y1="68.58" x2="50.8" y2="68.58" width="0.1524" layer="91"/>
@@
 <wire x1="-152.4" y1="-88.9" x2="-152.4" y2="-99.06" width="0.1524" layer="91"/>
 <label x="-152.4" y="-101.6" size="1.778" layer="95"/>
+</segment>
+<segment>
+<pinref part="U$3" gate="G$1" pin="-"/>
+<wire x1="-190.5" y1="71.12" x2="-190.5" y2="66.04" width="0.1524" layer="91"/>
+<label x="-190.5" y="66.04" size="1.778" layer="95"/>
 </segment>
 </net>
@@
 </segment>
 <segment>
-<pinref part="BOOSTER" gate="G$1" pin="2"/>
-<wire x1="60.96" y1="91.44" x2="53.34" y2="91.44" width="0.1524" layer="91"/>
-<label x="48.26" y="91.44" size="1.778" layer="95"/>
-</segment>
-<segment>
 <pinref part="REG5V" gate="G$1" pin="IN"/>
 <wire x1="-160.02" y1="78.74" x2="-165.1" y2="78.74" width="0.1524" layer="91"/>
@@
 <wire x1="60.96" y1="58.42" x2="53.34" y2="58.42" width="0.1524" layer="91"/>
 <wire x1="53.34" y1="58.42" x2="53.34" y2="66.04" width="0.1524" layer="91"/>
-<pinref part="BOOSTER" gate="G$1" pin="3"/>
 <wire x1="53.34" y1="66.04" x2="53.34" y2="76.2" width="0.1524" layer="91"/>
 <wire x1="53.34" y1="76.2" x2="53.34" y2="88.9" width="0.1524" layer="91"/>
-<wire x1="53.34" y1="88.9" x2="60.96" y2="88.9" width="0.1524" layer="91"/>
 <label x="43.18" y="63.5" size="1.778" layer="95"/>
 <pinref part="POWERCAP1" gate="G$1" pin="2"/>
@@
 <junction x="53.34" y="76.2"/>
 <junction x="53.34" y="66.04"/>
+<label x="53.34" y="91.44" size="1.778" layer="95"/>
 </segment>
 <segment>
@@
 </segment>
 </net>
-<net name="N$10" class="0">
-<segment>
-<pinref part="U$3" gate="G$1" pin="-"/>
-<wire x1="-190.5" y1="71.12" x2="-190.5" y2="66.04" width="0.1524" layer="91"/>
-<label x="-190.5" y="66.04" size="1.778" layer="95"/>
-</segment>
-</net>

Commit message: Electronics wip
Parts:
- added R10, R11, R12, R13, R14, R15, R7, R9: 3K, rhoban:RESISTANCE-R0805
- added U1: CD4051BM, rhoban:CD4051BM
- added X1, X2, X3, X4, X5: JST-XH-10-PIN-LONG-PAD, Rembrandt Electronics - JST XH Connectors v1-0:JST-XH-10-PIN-LONG-PAD
Connections:
- new net CS1: R7.2, U1.0
- new net CS2: R9.2, U1.1
- new net CS3: R10.2, U1.2
- new net CS4: R11.2, U1.3
- new net CS5: R12.2, U1.4
- new net CS6: R13.2, U1.5
- new net CS7: R14.2, U1.6
- new net CS8: R15.2, U1.7
- new net CSA1: U1.A
- new net CSA2: U1.B
- new net CSA3: U1.C
- net 3.3: now also R10.1, R11.1, R12.1, R13.1, R14.1, R15.1, R7.1, R9.1, U1.VDD
- net GND: now also U1.COM_OUT/IN, U1.INH, U1.VEE, U1.VSS

Commit message: Maxon controllers (wip)
Parts:
- added C1, C17, C18, C2, C3, C4, C5, C6: 15pF, rhoban:C_EU_22PF
- added ENC1, ENC2, ENC3, ENC4: LS7366RSO14, rhoban:LS7366RSO14
- added R16, R17, R19, R20, R22, R23, R25, R26, R28, R29: 1K, rhoban:RESISTANCE-R0805
- added R18, R21, R24, R27, R30: 24k, rhoban:RESISTANCE-R0805
- added U$6, U$7, U$8, U$9: MAXON380200, rhoban:MAXON380200
- added XTAL1, XTAL2, XTAL3, XTAL4: 40Mhz, rhoban:QUARTZ
- R5: value 36 -> 60
- U$10: value LS7366RSO14 -> MAXON380200; device rhoban:LS7366RSO14 -> rhoban:MAXON380200
Connections:
- new net INDEX: ENC1.INDEX/, ENC2.INDEX/, ENC3.INDEX/, ENC4.INDEX/
- new net M1_A: ENC1.A, X1-9.S
- new net M1_B: ENC1.B, X1-10.S
- new net M1_DIR: U$6.DIR
- new net M1_HALL1: U$6.HALL1, X1-6.S
- new net M1_HALL2: U$6.HALL2, X1-7.S
- new net M1_HALL3: U$6.HALL3, X1-8.S
- new net M1_SPEED: U$6.SPEED
- new net M1_W1: U$6.W1, X1-1.S
- new net M1_W2: U$6.W2, X1-2.S
- new net M1_W3: U$6.W3, X1-3.S
- new net M2_A: ENC2.A, X2-9.S
- new net M2_B: ENC2.B, X2-10.S
- new net M2_DIR: U$7.DIR
- new net M2_HALL1: U$7.HALL1, X2-6.S
- new net M2_HALL2: U$7.HALL2, X2-7.S
- new net M2_HALL3: U$7.HALL3, X2-8.S
- new net M2_SPEED: U$7.SPEED
- new net M2_W1: U$7.W1, X2-1.S
- new net M2_W2: U$7.W2, X2-2.S
- new net M2_W3: U$7.W3, X2-3.S
- new net M3_A: ENC3.A, X3-9.S
- new net M3_B: ENC3.B, X3-10.S
- new net M3_DIR: U$8.DIR
- new net M3_HALL1: U$8.HALL1, X3-6.S
- new net M3_HALL2: U$8.HALL2, X3-7.S
- new net M3_HALL3: U$8.HALL3, X3-8.S
- new net M3_SPEED: U$8.SPEED
- new net M3_W1: U$8.W1, X3-1.S
- new net M3_W2: U$8.W2, X3-2.S
- new net M3_W3: U$8.W3, X3-3.S
- new net M4_A: ENC4.A, X4-9.S
- new net M4_B: ENC4.B, X4-10.S
- new net M4_DIR: U$9.DIR
- new net M4_HALL1: U$9.HALL1, X4-6.S
- new net M4_HALL2: U$9.HALL2, X4-7.S
- new net M4_HALL3: U$9.HALL3, X4-8.S
- new net M4_SPEED: U$9.SPEED
- new net M4_W1: U$9.W1, X4-1.S
- new net M4_W2: U$9.W2, X4-2.S
- new net M4_W3: U$9.W3, X4-3.S
- new net M5_DIR: U$10.DIR
- new net M5_HALL1: U$10.HALL1, X5-6.S
- new net M5_HALL2: U$10.HALL2, X5-7.S
- new net M5_HALL3: U$10.HALL3
- new net M5_SPEED: U$10.SPEED
- new net M5_W1: U$10.W1, X5-1.S
- new net M5_W2: U$10.W2, X5-2.S
- new net M5_W3: U$10.W3, X5-3.S
- new net MISO: ENC1.MISO, ENC2.MISO, ENC3.MISO, ENC4.MISO
- new net MOSI: ENC1.MOSI, ENC2.MOSI, ENC3.MOSI, ENC4.MOSI
- new net MOTORS_EN: U$10.ENABLE, U$6.ENABLE, U$7.ENABLE, U$8.ENABLE, U$9.ENABLE
- new net MT_HALL3: X5-8.S
- new net N$10: R16.2, U$6.DIGIN1
- new net N$12: R17.2, U$6.DIGIN2
- new net N$13: C1.2, ENC2.FCK0, XTAL2.2
- new net N$14: C2.2, ENC2.FCKI, XTAL2.1
- new net N$15: R19.2, U$7.DIGIN1
- new net N$16: R18.2, U$6.CURRENT
- new net N$18: R20.2, U$7.DIGIN2
- new net N$19: C17.2, ENC1.FCK0, XTAL1.2
- new net N$20: C18.2, ENC1.FCKI, XTAL1.1
- new net N$21: R21.2, U$7.CURRENT
- new net N$22: C3.2, ENC3.FCK0, XTAL3.2
- new net N$23: C4.2, ENC3.FCKI, XTAL3.1
- new net N$24: R22.2, U$8.DIGIN1
- new net N$25: R23.2, U$8.DIGIN2
- new net N$26: R24.2, U$8.CURRENT
- new net N$27: C5.2, ENC4.FCK0, XTAL4.2
- new net N$28: C6.2, ENC4.FCKI, XTAL4.1
- new net N$29: R25.2, U$9.DIGIN1
- new net N$30: R26.2, U$9.DIGIN2
- new net N$31: R27.2, U$9.CURRENT
- new net N$32: R28.2, U$10.DIGIN1
- new net N$33: R29.2, U$10.DIGIN2
- new net N$34: R30.2, U$10.CURRENT
- new net SCK: ENC1.SCK, ENC2.SCK, ENC3.SCK, ENC4.SCK
- net CS1: now also ENC1.SS/
- net CS2: now also ENC2.SS/
- net CS3: now also ENC3.SS/
- net CS4: now also ENC4.SS/
- net GND: now also C1.1, C17.1, C18.1, C2.1, C3.1, C4.1, C5.1, C6.1, ENC1.VSS, ENC2.VSS, ENC3.VSS, ENC4.VSS, R16.1, R18.1, R19.1, R21.1, R22.1, R24.1, R25.1, R27.1, R28.1, R30.1, U$10.GND, U$6.GND, U$7.GND, U$8.GND, U$9.GND, X1-4.S, X2-4.S, X3-4.S, X4-4.S, X5-4.S
- net VCC: now also ENC1.VDD, ENC2.VDD, ENC3.VDD, ENC4.VDD, R17.1, R20.1, R23.1, R26.1, R29.1, U$10.VCC, U$6.VCC, U$7.VCC, U$8.VCC, U$9.VCC, X1-5.S, X2-5.S, X3-5.S, X4-5.S, X5-5.S; no longer R5.1
- net VIN: now also R5.1, U$10.VIN, U$6.VIN, U$7.VIN, U$8.VIN, U$9.VIN
Other:
- note added: "CS MUX"
- moved on the sheet: COM1, COM2, COM3, EMIT, R10, R11, R12, R13, R14, R15, R4, R5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

Commit message: Routing ready board
Parts:
- added R31: 1K, rhoban:RESISTANCE-R0805
- added R32, R33: 3K, rhoban:RESISTANCE-R0805
- added SOLENOID2: CONNEC_1X02BIG, rhoban:CONNEC_1X02BIG
- added T3: NPN_BC817,215, rhoban:NPN_BC817,215
- added U$11: TO-247A, to-247_n-channel_igbt:TO-247A
- renumbered SOLENOID to SOLENOID1
Connections:
- removed net KICK: MAPLE.3, R1.1, R2.1
- new net IRQ1: COM1.IRQ, MAPLE.23
- new net IRQ2: COM2.IRQ, MAPLE.24
- new net IRQ3: COM3.IRQ, MAPLE.25
- new net KICK1: MAPLE.7, R1.1, R2.1
- new net KICK2: MAPLE.6, R31.1, R32.1
- new net N$17: R31.2, T3.B
- new net N$35: R33.1, T3.C, U$11.G
- new net N$36: SOLENOID2.2, U$11.C
- net 3.3: now also COM1.CE, COM1.VCC, COM2.CE, COM2.VCC, COM3.CE, COM3.VCC, R32.2
- net CS5: now also COM1.CSN
- net CS6: now also COM2.CSN
- net CS7: now also COM3.CSN
- net CSA1: now also MAPLE.20
- net CSA2: now also MAPLE.21
- net CSA3: now also MAPLE.22
- net GND: now also COM1.GND, COM2.GND, COM3.GND, T3.E, U$11.E
- net INDEX: now also MAPLE.26
- net M1_DIR: now also MAPLE.13
- net M1_SPEED: now also MAPLE.3
- net M2_DIR: now also MAPLE.14
- net M2_SPEED: now also MAPLE.4
- net M3_DIR: now also MAPLE.17
- net M3_SPEED: now also MAPLE.5
- net M4_DIR: now also MAPLE.18
- net M4_SPEED: now also MAPLE.8
- net M5_DIR: now also MAPLE.19
- net M5_SPEED: now also MAPLE.9
- net MISO: now also COM1.MISO, COM2.MISO, COM3.MISO, MAPLE.29
- net MOSI: now also COM1.MOSI, COM2.MOSI, COM3.MOSI, MAPLE.28
- net SCK: now also COM1.SCK, COM2.SCK, COM3.SCK, MAPLE.30
- net VBOOST: now also SOLENOID2.1
- net VIN: now also R33.2
Other:
- note added: "MOTORS"
- note removed: "ENCODERS?"
- moved on the sheet: C1, C17, C18, C2, C3, C4, C5, C6, COM3, ENC1, ENC2, ENC3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
