File: electronics/brushless.brd (EAGLE design)
At the start: 34.3 x 56.2 mm, 63 parts, among them J1 USB_MINI-B_SMT, X1 JST-XH-10-PIN-LONG-PAD

Commit message: mos (wip)
Parts:
- added Q1, Q2, Q3, Q4, Q5, Q6: BUK7Y12-40E, transistor-power:SOT669
- R1, R10, R11, R12, R14, R15, R16, R17, R18, R19, R2, R20, R21, R22, R23, R24, R25, R3, R4, R5, R6, R7, R8, R9: device rhoban:R0805 -> SparkFun-Resistors:0805
- R28, R29, R35, R36, R39, R40, R48, R49, R50: device SparkFun-Passives:0805 -> SparkFun-Resistors:0805
- moved U$4 14.0 mm to (30.5, 8.26)
- moved ENC1 13.4 mm to (5.71, 8.26), turned to 180 degrees
- moved J1 13.3 mm to (29.2, 9.53)
- moved R29 12.8 mm to (23.5, 9.53)
- moved R35 12.8 mm to (23.5, 11.4)
- moved C12 11.2 mm to (3.17, 21.0), turned to 90 degrees
- moved C21 10.9 mm to (7.62, 24.8), turned to 180 degrees
- moved R28 10.5 mm to (23.5, 14.0), turned to 180 degrees
- moved R39 10.2 mm to (29.2, 16.5), turned to 180 degrees
- moved R49 10.2 mm to (32.4, 16.5), turned to 180 degrees
- moved BUT 9.55 mm to (32.4, 20.3)
- moved D4 9.55 mm to (26.0, 20.3)
- moved RESET 9.55 mm to (29.2, 20.3)
- moved R36 9.55 mm to (26.0, 24.1)
- moved R40 9.55 mm to (29.2, 24.1)
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Connections:
- net GND: now also Q2.1, Q2.2, Q2.3, Q4.1, Q4.2, Q4.3, Q6.1, Q6.2, Q6.3
- net N$1: now also Q1.4
- net N$2: now also Q3.4
- net N$3: now also Q2.4
- net N$6: now also Q4.4
- net N$7: now also Q5.4
- net N$9: now also Q6.4
- net U_PHASE: now also Q1.1, Q1.2, Q1.3, Q2.MB
- net V+: now also Q1.MB, Q3.MB, Q5.MB
- net V_PHASE: now also Q3.1, Q3.2, Q3.3, Q4.MB
- net W_PHASE: now also Q5.1, Q5.2, Q5.3, Q6.MB
Other:
- board size 34.3 x 56.2 mm -> 34.3 x 49.8 mm

Commit message: tweak
Parts:
- removed R20, R21, R22: 2K, SparkFun-Resistors:0805
- R23, R24, R25: value 3K -> 15K
- moved R23 25.4 mm to (31.8, 27.9), turned to 180 degrees
- moved R24 25.1 mm to (31.8, 30.5), turned to 180 degrees
- moved Q2 19.7 mm to (7.62, 50.2)
- moved Q4 19.7 mm to (17.1, 50.2)
- moved Q6 19.7 mm to (26.7, 50.2)
- moved R25 16.3 mm to (31.8, 33.0), turned to 180 degrees
- moved R19 12.9 mm to (27.3, 50.8)
- moved R16 12.7 mm to (17.8, 50.8)
- moved R15 12.5 mm to (8.26, 50.8)
- moved R2 12.1 mm to (10.2, 50.8)
- moved R4 12.1 mm to (19.7, 50.8)
- moved R6 12.1 mm to (29.2, 50.8)
- moved R18 3.81 mm to (27.9, 38.7)
- moved D3 3.18 mm to (33.0, 31.8)
- moved R11 3.18 mm to (27.3, 27.3)
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Connections:
- removed net HALL1: R20.2, X1.6
- removed net HALL2: R21.2, X1.7
- removed net HALL3: R22.2, X1.8
- net ENC_A: now also X1.3; no longer X1.9
- net ENC_B: now also X1.4; no longer X1.10
- net GND: now also X1.10; no longer X1.4
- net HALLU: now also X1.6; no longer R20.1
- net HALLV: now also X1.7; no longer R21.1
- net HALLW: now also X1.8; no longer R22.1
- net VCC: now also X1.2; no longer X1.5
- net V_PHASE: now also X1.5; no longer X1.2
- net W_PHASE: now also X1.9; no longer X1.3
Routing:
- net GND: track 0.00 -> 46.7 mm
- net V+: track 0.00 -> 35.3 mm
- net U_PHASE: track 0.00 -> 11.7 mm
- net V_PHASE: track 0.00 -> 11.5 mm
- net W_PHASE: track 0.00 -> 11.2 mm
Other:
- board size 34.3 x 49.8 mm -> 36.8 x 56.2 mm

Commit message: tweak2
Parts:
- moved J1 1.27 mm to (30.5, 9.53)
- turned UC1 to 270 degrees

Commit message: place
Parts:
- moved UC1 0.90 mm to (15.9, 19.7), turned to 90 degrees
- moved ENC1 0.64 mm to (5.71, 7.62), turned to 0 degrees

Commit message: up
Parts:
- R23, R24, R25: value 15K -> 10K
Changed lines of the file:
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@@
 <element name="U$5" library="rhoban" package="CONNEC_1X08" value="CONNEC_1X08" x="18.415" y="1.905"/>
 <element name="X1" library="Rembrandt Electronics - JST XH Connectors v1-0" package="JST-XH-10-PACKAGE-LONG-PAD" value="JST-XH-10-PIN-LONG-PAD" x="17.145" y="44.45"/>
-<element name="R23" library="SparkFun-Resistors" package="0805" value="15K" x="31.75" y="27.94" rot="MR180">
+<element name="R23" library="SparkFun-Resistors" package="0805" value="10K" x="31.75" y="27.94" rot="MR180">
 <attribute name="PROD_ID" value=" " x="31.75" y="27.94" size="1.778" layer="28" rot="MR180" display="off"/>
 <attribute name="VALUE" value=" " x="31.75" y="27.94" size="1.778" layer="28" rot="MR180" display="off"/>
 </element>
-<element name="R24" library="SparkFun-Resistors" package="0805" value="15K" x="31.75" y="30.48" rot="MR180">
+<element name="R24" library="SparkFun-Resistors" package="0805" value="10K" x="31.75" y="30.48" rot="MR180">
 <attribute name="PROD_ID" value=" " x="31.75" y="30.48" size="1.778" layer="28" rot="MR180" display="off"/>
 <attribute name="VALUE" value=" " x="31.75" y="30.48" size="1.778" layer="28" rot="MR180" display="off"/>
 </element>
-<element name="R25" library="SparkFun-Resistors" package="0805" value="15K" x="31.75" y="33.02" rot="MR180">
+<element name="R25" library="SparkFun-Resistors" package="0805" value="10K" x="31.75" y="33.02" rot="MR180">
 <attribute name="PROD_ID" value=" " x="31.75" y="33.02" size="1.778" layer="28" rot="MR180" display="off"/>
 <attribute name="VALUE" value=" " x="31.75" y="33.02" size="1.778" layer="28" rot="MR180" display="off"/>

Commit message: wip
Parts:
- moved XTAL1 19.1 mm to (1.27, 18.4), turned to 90 degrees
- moved C17 18.9 mm to (1.91, 25.4)
- moved R25 17.8 mm to (14.0, 32.4), flipped to the top, turned to 270 degrees
- moved C18 16.5 mm to (1.91, 11.4), turned to 180 degrees
- moved R24 15.4 mm to (16.5, 32.4), flipped to the top, turned to 270 degrees
- moved R23 13.5 mm to (19.1, 32.4), flipped to the top, turned to 270 degrees
- moved C21 13.1 mm to (20.3, 27.9), turned to 90 degrees
- moved C20 11.9 mm to (12.7, 27.9), turned to 270 degrees
- moved PROGRAM 11.7 mm to (19.7, 18.4)
- moved OSC 11.3 mm to (16.5, 27.9), turned to 0 degrees
- moved ENC1 10.2 mm to (6.99, 17.8), flipped to the bottom, turned to 90 degrees
- moved C12 10.0 mm to (12.7, 24.1), flipped to the bottom, turned to 180 degrees
- moved U$5 9.86 mm to (15.9, 11.4)
- moved D3 9.44 mm to (24.1, 28.6), flipped to the bottom
- moved R13 9.44 mm to (24.1, 24.1), flipped to the bottom
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Connections:
- net RX1: now also UC1.31
- net TX1: now also UC1.30
Routing:
- net U_PHASE: track 11.7 -> 14.4 mm
Other:
- board size 36.8 x 56.2 mm -> 35.5 x 46.7 mm

Commit message: bl wip
Parts:
- removed PROGRAM: CONNEC_1X066PADS, rhoban:6PADS
- removed XTAL1: 40Mhz, rhoban:HC49US
- added C4: 1nF, SparkFun-Passives:0805@1
- added OSC1: 40Mhz, SparkFun2:CRYSTAL-SMD-5X3
- added R20: 2K, SparkFun-Resistors:0805
- added R21: 3K, SparkFun-Resistors:0805
- added U$7: ACS712, rhoban:SO8
- moved C20 14.2 mm to (26.1, 32.7), turned to 180 degrees
- moved C7 13.2 mm to (21.0, 15.6), turned to 270 degrees
- moved R36 13.1 mm to (23.3, 20.2)
- moved R25 12.1 mm to (23.5, 39.9), turned to 90 degrees
- moved C12 11.4 mm to (1.27, 24.8)
- moved OSC 9.65 mm to (26.1, 28.9), turned to 270 degrees
- moved R50 8.95 mm to (32.3, 19.8), turned to 270 degrees
- moved R24 8.70 mm to (21.0, 39.9), turned to 90 degrees
- moved R23 8.38 mm to (17.9, 40.7), turned to 0 degrees
- moved R28 6.86 mm to (30.4, 19.8), turned to 90 degrees
- moved R40 6.80 mm to (30.0, 26.3), turned to 90 degrees
- moved D4 6.54 mm to (25.7, 22.7), turned to 0 degrees
- moved C21 6.45 mm to (26.1, 25.1), turned to 0 degrees
- moved UC1 5.97 mm to (12.1, 24.3), turned to 90 degrees
- moved RESET 5.86 mm to (32.9, 24.6)
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Connections:
- new net CUR: R20.2, R21.1, UC1.17
- new net N$24: R20.1, U$7.7
- new net N$27: C4.1, U$7.6
- new net V+_MOS: Q1.MB, Q3.MB, Q5.MB, U$7.1, U$7.2
- net 3.3: no longer PROGRAM.2
- net BOOT1: no longer PROGRAM.4
- net GND: now also C4.2, R21.2, U$7.5; no longer PROGRAM.1
- net N$20: now also OSC1.1; no longer XTAL1.2
- net N$21: now also OSC1.3; no longer XTAL1.1
- net RESET: no longer PROGRAM.3
- net RX1: no longer PROGRAM.6
- net TX1: no longer PROGRAM.5
- net V+: now also U$7.3, U$7.4; no longer Q1.MB, Q3.MB, Q5.MB
- net VCC: now also U$7.8
Routing:
- net V+_MOS: track 0.00 -> 25.2 mm
- net V+: track 35.3 -> 15.3 mm
- net GND: track 46.7 -> 47.9 mm

Commit message: wip
Parts:
- moved ENC1 19.3 mm to (9.86, 37.2), flipped to the top, turned to 0 degrees
- moved C18 17.9 mm to (9.80, 30.3), flipped to the top, turned to 90 degrees
- moved C21 14.2 mm to (12.9, 19.9), turned to 270 degrees
- moved C20 14.0 mm to (20.5, 19.9), turned to 90 degrees
- moved R13 13.5 mm to (31.9, 20.9), turned to 0 degrees
- moved OSC 13.0 mm to (16.7, 19.9), turned to 180 degrees
- moved OSC1 12.9 mm to (5.99, 30.3), flipped to the top, turned to 0 degrees
- moved C7 11.2 mm to (10.6, 19.9)
- moved D4 9.37 mm to (25.5, 32.1), turned to 90 degrees
- moved C17 8.39 mm to (2.18, 30.3), flipped to the top, turned to 270 degrees
- moved U$4 7.98 mm to (22.2, 19.2)
- moved R36 7.67 mm to (25.5, 27.6), turned to 90 degrees
- moved D3 7.37 mm to (26.4, 28.3)
- moved D1 7.32 mm to (8.59, 28.3)
- moved D2 7.32 mm to (17.5, 28.3)
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Other:
- board size 35.5 x 46.7 mm -> 35.5 x 43.3 mm
